Commit message: Get arm building

File: sawyer_description/urdf/sawyer.urdf.xacro (robot description, xacro)
@@ -5,20 +5,16 @@
   <xacro:arg name="static" default="true"/>
   <xacro:arg name="electric_gripper" default="false"/>
+  <xacro:property name="gazebo" value="$(arg gazebo)"/>
+  <xacro:property name="pedestal" value="$(arg pedestal)"/>
+  <xacro:property name="static" value="$(arg static)"/>
+  <xacro:property name="electric_gripper" value="$(arg electric_gripper)"/>
   <!-- Sawyer Base URDF -->
-  <xacro:include filename="$(find sawyer_description)/urdf/sawyer_base.urdf.xacro">
-    <xacro:arg name="gazebo" value="${gazebo}"/>
-    <xacro:arg name="pedestal" value="${pedestal}"/>
-  </xacro:include>
-  <xacro:if value="$(arg gazebo)">
-  <xacro:include filename="$(find sawyer_description)/urdf/sawyer_base.gazebo.xacro">
-    <xacro:arg name="static" value="${static}"/>
-    <xacro:arg name="pedestal" value="${pedestal}"/>
-  </xacro:include>
+  <xacro:include filename="$(find sawyer_description)/urdf/sawyer_base.urdf.xacro"/>
+  <xacro:if value="${gazebo}">
+    <xacro:include filename="$(find sawyer_description)/urdf/sawyer_base.gazebo.xacro"/>
   </xacro:if>
   <!-- Electric Gripper End Effector -->
   <xacro:if value="$(arg electric_gripper)">
-  <xacro:include filename="$(find sawyer_description)/urdf/sawyer_electric_gripper.urdf.xacro">
-    <xacro:arg name="gazebo" value="${gazebo}"/>
-  </xacro:include>
+    <xacro:include filename="$(find sawyer_description)/urdf/sawyer_electric_gripper.urdf.xacro"/>
   </xacro:if>
 </robot>

File: sawyer_description/urdf/sawyer_base.urdf.xacro (robot description, xacro)
@@ -42,5 +42,5 @@
       <origin rpy="1.57079632679 0 -1.57079632679" xyz="0.26 0.345 -0.91488"/>
       <geometry>
-        <mesh filename="package://sawyer_description/meshes/sawyer_pv/pedestal.DAE"/>
+        <mesh filename="file://$(find sawyer_description)/meshes/sawyer_pv/pedestal.DAE"/>
       </geometry>
       <material name="darkgray"/>
@@ -109,5 +109,5 @@
       <origin rpy="0 0 0" xyz="0 0 0"/>
       <geometry>
-        <mesh filename="package://sawyer_description/meshes/sawyer_pv/base.DAE"/>
+        <mesh filename="file://$(find sawyer_description)/meshes/sawyer_pv/base.DAE"/>
       </geometry>
       <material name="sawyer_red"/>
@@ -129,5 +129,5 @@
       <origin rpy="0 0 0" xyz="0 0 0"/>
       <geometry>
-        <mesh filename="package://sawyer_description/meshes/sawyer_mp3/l0.DAE"/>
+        <mesh filename="file://$(find sawyer_description)/meshes/sawyer_mp3/l0.DAE"/>
       </geometry>
       <material name="sawyer_red"/>
@@ -159,5 +159,5 @@
       <origin rpy="0 0 0" xyz="0 0 0"/>
       <geometry>
-        <mesh filename="package://sawyer_description/meshes/sawyer_pv/head.DAE"/>
+        <mesh filename="file://$(find sawyer_description)/meshes/sawyer_pv/head.DAE"/>
       </geometry>
       <material name="sawyer_red"/>
@@ -204,5 +204,5 @@
       <origin rpy="0 0 0" xyz="0 0 0"/>
       <geometry>
-        <mesh filename="package://sawyer_description/meshes/sawyer_mp3/l1.DAE"/>
+        <mesh filename="file://$(find sawyer_description)/meshes/sawyer_mp3/l1.DAE"/>
       </geometry>
       <material name="sawyer_red"/>
@@ -234,5 +234,5 @@
       <origin rpy="0 0 0" xyz="0 0 0"/>
       <geometry>
-        <mesh filename="package://sawyer_description/meshes/sawyer_pv/l2.DAE"/>
+        <mesh filename="file://$(find sawyer_description)/meshes/sawyer_pv/l2.DAE"/>
       </geometry>
       <material name="sawyer_red"/>
@@ -264,5 +264,5 @@
       <origin rpy="0 0 0" xyz="0 0 0"/>
       <geometry>
-        <mesh filename="package://sawyer_description/meshes/sawyer_pv/l3.DAE"/>
+        <mesh filename="file://$(find sawyer_description)/meshes/sawyer_pv/l3.DAE"/>
       </geometry>
       <material name="sawyer_red"/>
@@ -294,5 +294,5 @@
       <origin rpy="0 0 0" xyz="0 0 0"/>
       <geometry>
-        <mesh filename="package://sawyer_description/meshes/sawyer_pv/l4.DAE"/>
+        <mesh filename="file://$(find sawyer_description)/meshes/sawyer_pv/l4.DAE"/>
       </geometry>
       <material name="sawyer_red"/>
@@ -339,5 +339,5 @@
       <origin rpy="0 0 0" xyz="0 0 0"/>
       <geometry>
-        <mesh filename="package://sawyer_description/meshes/sawyer_pv/l5.DAE"/>
+        <mesh filename="file://$(find sawyer_description)/meshes/sawyer_pv/l5.DAE"/>
       </geometry>
       <material name="sawyer_red"/>
@@ -383,5 +383,5 @@
       <origin rpy="0 0 0" xyz="0 0 0"/>
       <geometry>
-        <mesh filename="package://sawyer_description/meshes/sawyer_mp1/l6.DAE"/>
+        <mesh filename="file://$(find sawyer_description)/meshes/sawyer_mp1/l6.DAE"/>
       </geometry>
       <material name="sawyer_red"/>
